Commit message: Reduced number of links in tether for testing

File: sdf_models/models/tether/model.urdf (robot description, URDF)
Before this commit: robot tether, 12 links, 11 joints
Links:
- removed link element_10
- removed link element_11
- removed link element_3
- removed link element_4
- removed link element_5
- removed link element_6
- removed link element_7
- removed link element_8
- removed link element_9
- link element_0: mass 0.0006666666666666666 -> 0.0006666666666666668
- link element_1: mass 0.01 -> 0.1; geometry collision cylinder length=0.0001 radius=0.0001; visual cylinder length=1.5 radius=0.01
- link element_2: mass 0.01 -> 0.0006666666666666668; geometry collision cylinder length=0.0001 radius=0.0001; visual cylinder length=0.01 radius=0.01
Joints:
- removed joint joint_10_to_11
- removed joint joint_2_to_3
- removed joint joint_3_to_4
- removed joint joint_4_to_5
- removed joint joint_5_to_6
- removed joint joint_6_to_7
- removed joint joint_7_to_8
- removed joint joint_8_to_9
- removed joint joint_9_to_10
- joint joint_1_to_2: origin xyz=0.15 0 0 rpy=0 0 0 -> xyz=1.5 0 0 rpy=0 0 0

File: sdf_models/models/tether/model.xacro (robot description, xacro)
@@ -8,5 +8,5 @@
     <xacro:property name="tether_radius" value="0.01" />
     <xacro:property name="tether_mass" value="0.1" />
-    <xacro:property name="num_elements" value="10" />
+    <xacro:property name="num_elements" value="1" />
     <xacro:property name="elem_length_main" value="${tether_length/num_elements}" />
     <xacro:property name="elem_length_ends" value="0.01" />

Commit message: Can specify initial drone + tether pose

File: sdf_models/models/tether/model.urdf (robot description, URDF)
Before this commit: robot tether, 3 links, 2 joints
Links:
- removed link element_0
- removed link element_2
Joints:
- removed joint joint_0_to_1
- removed joint joint_1_to_2

File: sdf_models/models/tether/model.xacro (robot description, xacro)
@@ -10,7 +10,7 @@
     <xacro:property name="num_elements" value="1" />
     <xacro:property name="elem_length_main" value="${tether_length/num_elements}" />
-    <xacro:property name="elem_length_ends" value="0.01" />
+    <!-- <xacro:property name="elem_length_ends" value="0.01" /> -->
     <xacro:property name="elem_mass_main" value="${tether_mass/num_elements}" />
-    <xacro:property name="elem_mass_ends" value="${elem_mass_main*(elem_length_ends/elem_length_main)}" />
+    <!-- <xacro:property name="elem_mass_ends" value="${elem_mass_main*(elem_length_ends/elem_length_main)}" /> -->
     <!-- Define link macro -->
     <xacro:macro name="tether_element" params="element_num elem_length elem_mass">
@@ -62,7 +62,7 @@
     <xacro:generate_tether elem_num="${num_elements}" />
     <!-- Add start and end elements and joints-->
-    <xacro:tether_element element_num="0" elem_length="${elem_length_ends}" elem_mass="${elem_mass_ends}" />
-    <xacro:tether_element element_num="${num_elements+1}" elem_length="${elem_length_ends}" elem_mass="${elem_mass_ends}" />
-    <joint name="joint_0_to_1" type="continuous">
+    <!-- <xacro:tether_element element_num="0" elem_length="${elem_length_ends}" elem_mass="${elem_mass_ends}" />
+    <xacro:tether_element element_num="${num_elements+1}" elem_length="${elem_length_ends}" elem_mass="${elem_mass_ends}" /> -->
+    <!-- <joint name="joint_0_to_1" type="continuous">
         <axis xyz="0. 1. 1."/>
         <origin xyz="${elem_length_ends} 0 0" rpy="0 0 0"/>
@@ -75,5 +75,5 @@
         <parent link="element_${num_elements}"/>
         <child link="element_${num_elements+1}"/>
-    </joint>
+    </joint> -->
     <!-- Define joints -->
         <!-- Add start element joint-->
