Commit message: Commit before video. Mucking with x500 SDF

File: sdf_models/models/tether/model.xacro (robot description, xacro)
@@ -7,5 +7,5 @@
     <xacro:property name="tether_length" value="1.5" />
     <xacro:property name="tether_radius" value="0.01" />
-    <xacro:property name="tether_mass" value="0.1" />
+    <xacro:property name="tether_mass" value="0.001" />
     <xacro:property name="num_elements" value="1" />
     <xacro:property name="elem_length_main" value="${tether_length/num_elements}" />
